File: RadioReceiver/RadioReceiver.kicad_sch (KiCad schematic)
At the start: 45 parts

Commit message: Add Linux/macOS support and self-contained project libraries
- Scripts: Add platform detection for KiCAD paths (Linux/macOS/Windows)
- enrich_parts.py: Switch to official JLCPCB BOM API
- assign_designators.py: Add duplicate validation, auto-select first option
- parse_library_pins.py: Extract LCSC codes from symbols
- map_connections.py: Remove hardcoded mappings, derive from symbol_pins.json
- Libraries: Copy JLCPCB symbols/footprints/3D models into project
- Library tables: Use ${KIPRJMOD} relative paths for portability
- Part substitutions: TS-1102S -> TS-1187A-B-A-B, PJ-327A -> PJ-3537S-SMT

🤖 Generated with [Claude Code](https://claude.com/claude-code)

Co-Authored-By: Claude Opus 4.5 <noreply@anthropic.com>
Parts:
- removed ANT1: (no value), symbol JLCPCB:FM_Wire
- removed ANT2: (no value), symbol JLCPCB:AM_Loop
- removed C1, C2, C3: (no value), symbol JLCPCB:CL21A106KOQNNNE
- removed C10, C11, C12, C13, C14, C15, C16, C6, C7, C8, C9: (no value), symbol JLCPCB:CL10B104KB8NNNC
- removed C4, C5: (no value), symbol JLCPCB:CL21A226MQQNNNE
- removed D4, D5: (no value), symbol JLCPCB:BSP752R
- removed J1: (no value), symbol JLCPCB:TYPE-C16PIN
- removed J3: (no value), symbol JLCPCB:PJ-227-5A
- removed R3: (no value), symbol JLCPCB:RMC06032K5%N
- removed R4: (no value), symbol JLCPCB:RMC_0603_10K_J_N
- removed SW1: (no value), symbol JLCPCB:K2-1102SP-C4SC-04
- removed Y1: (no value), symbol JLCPCB:Q13FC1350000400
- added ANT1, ANT2: (no value), DNP, symbol DNP
- added C1, C2, C3: (no value), symbol JLCPCB:CL21A106KAYNNNE
- added C10, C11, C12, C13, C14, C15, C16, C6, C7, C8, C9: (no value), symbol JLCPCB:CC0603KRX7R9BB104
- added C4, C5: (no value), symbol JLCPCB:CL21A226MAQNNNE
- added D4, D5: (no value), symbol JLCPCB:AP1501-50K5G-13
- added J1: (no value), symbol JLCPCB:TYPE-C-31-M-12
- added J3: (no value), symbol JLCPCB:PJ-3537S
- added R3: (no value), symbol JLCPCB:0603WAF2001T5E
- added R4: (no value), symbol JLCPCB:0603WAF1002T5E
- added SW1: (no value), symbol JLCPCB:TS-1187A-B-A-B
- added Y1: (no value), symbol JLCPCB:X206032768KGB2SC
- U4: LCSC C195417 -> C1526089
